Commit message: #6 Fix lidar operation

File: vehicle_ws/src/diff_drive/description/diffbot.xacro (robot description, xacro)
@@ -1,4 +1,4 @@
 <?xml version='1.0'?>
-<robot name="slambot" xmlns:xacro="http://www.ros.org/wiki/xacro">
+<robot name="diffbot" xmlns:xacro="http://www.ros.org/wiki/xacro">
   <!-- LINK: base_footprint -->
   <link name="base_footprint"></link>
@@ -9,5 +9,5 @@
       <mass value="15.0"/>
       <origin xyz="0 0 0" rpy=" 0 0 0"/>
-      <inertia ixx="0.1" ixy="0" ixz="0" iyy="0.1" iyz="0" izz="0.1" />
+      <inertia ixx="0.1" ixy="0" ixz="0" iyy="0.1" iyz="0" izz="0.1"/>
     </inertial>
     <collision name='chassis_collision'>
@@ -29,5 +29,5 @@
       <mass value="8.0"/>
       <origin xyz="0 0 0" rpy=" 0 1.5707 1.5707"/>
-      <inertia ixx="0.1" ixy="0" ixz="0" iyy="0.1" iyz="0" izz="0.1" />
+      <inertia ixx="0.1" ixy="0" ixz="0" iyy="0.1" iyz="0" izz="0.1"/>
     </inertial>
     <collision>
@@ -49,5 +49,5 @@
       <mass value="8.0"/>
       <origin xyz="0 0 0" rpy=" 0 1.5707 1.5707"/>
-      <inertia ixx="0.1" ixy="0" ixz="0" iyy="0.1" iyz="0" izz="0.1" />
+      <inertia ixx="0.1" ixy="0" ixz="0" iyy="0.1" iyz="0" izz="0.1"/>
     </inertial>
     <collision>
@@ -69,5 +69,5 @@
       <mass value="8.0"/>
       <origin xyz="0 0 0" rpy=" 0 1.5707 1.5707"/>
-      <inertia ixx="0.1" ixy="0" ixz="0" iyy="0.1" iyz="0" izz="0.1" />
+      <inertia ixx="0.1" ixy="0" ixz="0" iyy="0.1" iyz="0" izz="0.1"/>
     </inertial>
     <collision>
@@ -89,5 +89,5 @@
       <mass value="8.0"/>
       <origin xyz="0 0 0" rpy=" 0 1.5707 1.5707"/>
-      <inertia ixx="0.1" ixy="0" ixz="0" iyy="0.1" iyz="0" izz="0.1" />
+      <inertia ixx="0.1" ixy="0" ixz="0" iyy="0.1" iyz="0" izz="0.1"/>
     </inertial>
     <collision>
@@ -109,10 +109,10 @@
       <mass value="1e-5"/>
       <origin xyz="0 0 0" rpy=" 0 0 0"/>
-      <inertia ixx="1e-6" ixy="0" ixz="0" iyy="1e-6" iyz="0" izz="1e-6" />
+      <inertia ixx="1e-6" ixy="0" ixz="0" iyy="1e-6" iyz="0" izz="1e-6"/>
     </inertial>
     <visual name="hokuyo_visual">
       <origin xyz="0 0 0" rpy="0 0 0" />
       <geometry>
-        <box size="0.05 0.05 0.05"/>
+        <cylinder length="0.15" radius="0.1"/>
       </geometry>
     </visual>
@@ -120,5 +120,5 @@
       <origin xyz="0 0 0" rpy="0 0 0" />
       <geometry>
-        <box size="0.1 0.1 0.1"/>
+        <cylinder length="0.15" radius="0.1"/>
       </geometry>
     </collision>
@@ -126,7 +126,7 @@
   <!-- JOINT: chassis -->
   <joint name="chassis_joint" type="fixed">
-    <origin xyz="0 0 0" rpy="0 0 0" />
-    <parent link="base_footprint"/>
-    <child link="chassis" />
+    <origin xyz="0 0 0" rpy="0 0 0"/>
+    <parent link="base_footprint"/>
+    <child link="chassis"/>
   </joint>
   <!-- JOINT: wheel -->
@@ -168,8 +168,8 @@
   <!-- JOINT: hokuyo -->
   <joint type="fixed" name="hokuyo_joint">
-    <origin xyz="0.15 0 0.3" rpy="0 0 0"/>
+    <origin xyz="0 0 0.125" rpy="0 0 0"/>
     <child link="hokuyo"/>
     <parent link="base_footprint"/>
-    <axis xyz="0 1 0" rpy="0 0 0"/>
+    <axis xyz="0 0 1" rpy="0 0 0"/>
   </joint>
   <!-- COLOR: chassis -->
@@ -219,5 +219,5 @@
       <max_wheel_torque>15</max_wheel_torque>
       <publish_odom>true</publish_odom>
-      <publish_odom_tf>true</publish_odom_tf>
+      <publish_odom_tf>false</publish_odom_tf>
       <publish_wheel_tf>false</publish_wheel_tf>
     </plugin>
@@ -227,5 +227,5 @@
     <sensor type="ray" name="head_hokuyo_sensor">
       <pose>0 0 0 0 0 0</pose>
-      <visualize>false</visualize>
+      <visualize>true</visualize>
       <update_rate>40</update_rate>
       <ray>
@@ -239,5 +239,5 @@
         </scan>
         <range>
-          <min>0.10</min>
+          <min>0.15</min>
           <max>30.0</max>
           <resolution>0.01</resolution>

Commit message: #6 Configure lidar

File: vehicle_ws/src/diff_drive/description/diffbot.xacro (robot description, xacro)
@@ -104,6 +104,6 @@
     </visual>
   </link>
-  <!-- LINK: hokuyo -->
-  <link name="hokuyo">
+  <!-- LINK: lidar -->
+  <link name="lidar">
     <inertial>
       <mass value="1e-5"/>
@@ -111,5 +111,5 @@
       <inertia ixx="1e-6" ixy="0" ixz="0" iyy="1e-6" iyz="0" izz="1e-6"/>
     </inertial>
-    <visual name="hokuyo_visual">
+    <visual name="lidar_visual">
       <origin xyz="0 0 0" rpy="0 0 0" />
       <geometry>
@@ -117,5 +117,5 @@
       </geometry>
     </visual>
-    <collision name="hokuyo_colision">
+    <collision name="lidar_colision">
       <origin xyz="0 0 0" rpy="0 0 0" />
       <geometry>
@@ -166,8 +166,8 @@
     <dynamics damping="1.0" friction="1.0"/>
   </joint>
-  <!-- JOINT: hokuyo -->
-  <joint type="fixed" name="hokuyo_joint">
+  <!-- JOINT: lidar -->
+  <joint type="fixed" name="lidar_joint">
     <origin xyz="0 0 0.125" rpy="0 0 0"/>
-    <child link="hokuyo"/>
+    <child link="lidar"/>
     <parent link="base_footprint"/>
     <axis xyz="0 0 1" rpy="0 0 0"/>
@@ -193,6 +193,6 @@
     <material>Gazebo/Grey</material>
   </gazebo>
-  <!-- COLOR: hokuyo -->
-  <gazebo reference="hokuyo">
+  <!-- COLOR: lidar -->
+  <gazebo reference="lidar">
     <material>Gazebo/Black</material>
   </gazebo>
@@ -224,13 +224,13 @@
   </gazebo>
   <!-- PLUGIN: sensor -->
-  <gazebo reference="hokuyo">
-    <sensor type="ray" name="head_hokuyo_sensor">
+  <gazebo reference="lidar">
+    <sensor type="ray" name="lidar_sensor">
       <pose>0 0 0 0 0 0</pose>
-      <visualize>true</visualize>
+      <visualize>false</visualize>
       <update_rate>40</update_rate>
       <ray>
         <scan>
           <horizontal>
-            <samples>720</samples>
+            <samples>600</samples>
             <resolution>1</resolution>
             <min_angle>-3.141592</min_angle>
@@ -240,5 +240,5 @@
         <range>
           <min>0.15</min>
-          <max>30.0</max>
+          <max>10.0</max>
           <resolution>0.01</resolution>
         </range>
@@ -255,5 +255,4 @@
         </ros>
         <output_type>sensor_msgs/LaserScan</output_type>
-        <namespace>/diffbot</namespace>
       </plugin>
     </sensor>
