Commit message: #8 Piracer assembly

File: piracer_ws/src/digital_twin/description/piracer.xacro (robot description, xacro)
@@ -24,4 +24,46 @@
     </visual>
   </link>
+  <!-- LINK: left_steer -->
+  <link name="left_steer">
+    <pose>0 0 0 0 0 0</pose>
+    <inertial>
+      <mass value="0.1"/>
+      <origin xyz="0 0 0" rpy="0 0 0"/>
+      <inertia ixx="0.1" ixy="0" ixz="0" iyy="0.1" iyz="0" izz="0.1"/>
+    </inertial>
+    <collision name="left_steer_collision">
+      <origin xyz="0 0 0" rpy="0 0 0"/>
+      <geometry>
+        <cylinder length="0.022" radius="0.002"/>
+      </geometry>
+    </collision>
+    <visual name="left_steer_visual">
+      <origin xyz="0 0 0" rpy="0 0 0"/>
+      <geometry>
+        <cylinder length="0.022" radius="0.002"/>
+      </geometry>
+    </visual>
+  </link>
+  <!-- LINK: right_steer -->
+  <link name="right_steer">
+    <pose>0 0 0 0 0 0</pose>
+    <inertial>
+      <mass value="0.1"/>
+      <origin xyz="0 0 0" rpy="0 0 0"/>
+      <inertia ixx="0.1" ixy="0" ixz="0" iyy="0.1" iyz="0" izz="0.1"/>
+    </inertial>
+    <collision name="right_steer_collision">
+      <origin xyz="0 0 0" rpy="0 0 0"/>
+      <geometry>
+        <cylinder length="0.022" radius="0.002"/>
+      </geometry>
+    </collision>
+    <visual name="right_steer_visual">
+      <origin xyz="0 0 0" rpy="0 0 0"/>
+      <geometry>
+        <cylinder length="0.022" radius="0.002"/>
+      </geometry>
+    </visual>
+  </link>
   <!-- LINK: board -->
   <link name="board">
@@ -40,5 +82,5 @@
     </visual>
   </link>
-  <!-- LINK: board -->
+  <!-- LINK: rpi -->
   <link name="rpi">
     <pose>0 0 0 0 0 0</pose>
@@ -53,4 +95,200 @@
       <geometry>
         <mesh scale="0.001 0.001 0.001" filename="package://digital_twin/meshes/rpi.stl"/>
+      </geometry>
+    </visual>
+  </link>
+  <!-- LINK: motor1 -->
+  <link name="motor1">
+    <pose>0 0 0 0 0 0</pose>
+    <collision name="motor1_collision">
+      <origin xyz="0 0 0" rpy="0 0 0"/>
+      <geometry>
+        <mesh scale="0.001 0.001 0.001" filename="package://digital_twin/meshes/motor.stl"/>
+      </geometry>
+    </collision>
+    <visual name="motor1_visual">
+      <origin xyz="0 0 0" rpy="0 0 0"/>
+      <geometry>
+        <mesh scale="0.001 0.001 0.001" filename="package://digital_twin/meshes/motor.stl"/>
+      </geometry>
+    </visual>
+  </link>
+  <!-- LINK: motor2 -->
+  <link name="motor2">
+    <pose>0 0 0 0 0 0</pose>
+    <collision name="motor2_collision">
+      <origin xyz="0 0 0" rpy="0 0 0"/>
+      <geometry>
+        <mesh scale="0.001 0.001 0.001" filename="package://digital_twin/meshes/motor.stl"/>
+      </geometry>
+    </collision>
+    <visual name="motor2_visual">
+      <origin xyz="0 0 0" rpy="0 0 0"/>
+      <geometry>
+        <mesh scale="0.001 0.001 0.001" filename="package://digital_twin/meshes/motor.stl"/>
+      </geometry>
+    </visual>
+  </link>
+  <!-- LINK: cover -->
+  <link name="cover">
+    <pose>0 0 0 0 0 0</pose>
+    <collision name="cover_collision">
+      <origin xyz="0 0 0" rpy="0 0 0"/>
+      <geometry>
+        <mesh scale="0.001 0.001 0.001" filename="package://digital_twin/meshes/cover.stl"/>
+      </geometry>
+    </collision>
+    <visual name="cover_visual">
+      <origin xyz="0 0 0" rpy="0 0 0"/>
+      <geometry>
+        <mesh scale="0.001 0.001 0.001" filename="package://digital_twin/meshes/cover.stl"/>
+      </geometry>
+    </visual>
+  </link>
+  <!-- LINK: rear_left_tire -->
+  <link name="rear_left_tire">
+    <pose>0 0 0 0 0 0</pose>
+    <inertial>
+      <mass value="1.0"/>
+      <origin xyz="0 0 0" rpy="0 0 0"/>
+      <inertia ixx="0.1" ixy="0" ixz="0" iyy="0.1" iyz="0" izz="0.1"/>
+    </inertial>
+    <collision name="rear_left_tire_collision">
+      <origin xyz="0 0 0" rpy="0 0 0"/>
+      <geometry>
+        <mesh scale="0.001 0.001 0.001" filename="package://digital_twin/meshes/tire.stl"/>
+      </geometry>
+    </collision>
+    <visual name="rear_left_tire_visual">
+      <origin xyz="0 0 0" rpy="0 0 0"/>
+      <geometry>
+        <mesh scale="0.001 0.001 0.001" filename="package://digital_twin/meshes/tire.stl"/>
+      </geometry>
+    </visual>
+  </link>
+  <!-- LINK: rear_left_disk -->
+  <link name="rear_left_disk">
+    <pose>0 0 0 0 0 0</pose>
+    <collision name="rear_left_disk_collision">
+      <origin xyz="0 0 0" rpy="0 0 0"/>
+      <geometry>
+        <mesh scale="0.001 0.001 0.001" filename="package://digital_twin/meshes/disk.stl"/>
+      </geometry>
+    </collision>
+    <visual name="rear_left_disk_visual">
+      <origin xyz="0 0 0" rpy="0 0 0"/>
+      <geometry>
+        <mesh scale="0.001 0.001 0.001" filename="package://digital_twin/meshes/disk.stl"/>
+      </geometry>
+    </visual>
+  </link>
+  <!-- LINK: rear_right_tire -->
+  <link name="rear_right_tire">
+    <pose>0 0 0 0 0 0</pose>
+    <inertial>
+      <mass value="1.0"/>
+      <origin xyz="0 0 0" rpy="0 0 0"/>
+      <inertia ixx="0.1" ixy="0" ixz="0" iyy="0.1" iyz="0" izz="0.1"/>
+    </inertial>
+    <collision name="rear_right_tire_collision">
+      <origin xyz="0 0 0" rpy="0 0 0"/>
+      <geometry>
+        <mesh scale="0.001 0.001 0.001" filename="package://digital_twin/meshes/tire.stl"/>
+      </geometry>
+    </collision>
+    <visual name="rear_right_tire_visual">
+      <origin xyz="0 0 0" rpy="0 0 0"/>
+      <geometry>
+        <mesh scale="0.001 0.001 0.001" filename="package://digital_twin/meshes/tire.stl"/>
+      </geometry>
+    </visual>
+  </link>
+  <!-- LINK: rear_right_disk -->
+  <link name="rear_right_disk">
+    <pose>0 0 0 0 0 0</pose>
+    <collision name="rear_right_disk_collision">
+      <origin xyz="0 0 0" rpy="0 0 0"/>
+      <geometry>
+        <mesh scale="0.001 0.001 0.001" filename="package://digital_twin/meshes/disk.stl"/>
+      </geometry>
+    </collision>
+    <visual name="rear_right_disk_visual">
+      <origin xyz="0 0 0" rpy="0 0 0"/>
+      <geometry>
+        <mesh scale="0.001 0.001 0.001" filename="package://digital_twin/meshes/disk.stl"/>
+      </geometry>
+    </visual>
+  </link>
+  <!-- LINK: front_left_tire -->
+  <link name="front_left_tire">
+    <pose>0 0 0 0 0 0</pose>
+    <inertial>
+      <mass value="1.0"/>
+      <origin xyz="0 0 0" rpy="0 0 0"/>
+      <inertia ixx="0.1" ixy="0" ixz="0" iyy="0.1" iyz="0" izz="0.1"/>
+    </inertial>
+    <collision name="front_left_tire_collision">
+      <origin xyz="0 0 0" rpy="0 0 0"/>
+      <geometry>
+        <mesh scale="0.001 0.001 0.001" filename="package://digital_twin/meshes/tire.stl"/>
+      </geometry>
+    </collision>
+    <visual name="front_left_tire_visual">
+      <origin xyz="0 0 0" rpy="0 0 0"/>
+      <geometry>
+        <mesh scale="0.001 0.001 0.001" filename="package://digital_twin/meshes/tire.stl"/>
+      </geometry>
+    </visual>
+  </link>
+  <!-- LINK: front_left_disk -->
+  <link name="front_left_disk">
+    <pose>0 0 0 0 0 0</pose>
+    <collision name="front_left_disk_collision">
+      <origin xyz="0 0 0" rpy="0 0 0"/>
+      <geometry>
+        <mesh scale="0.001 0.001 0.001" filename="package://digital_twin/meshes/disk.stl"/>
+      </geometry>
+    </collision>
+    <visual name="front_left_disk_visual">
+      <origin xyz="0 0 0" rpy="0 0 0"/>
+      <geometry>
+        <mesh scale="0.001 0.001 0.001" filename="package://digital_twin/meshes/disk.stl"/>
+      </geometry>
+    </visual>
+  </link>
+  <!-- LINK: front_right_tire -->
+  <link name="front_right_tire">
+    <pose>0 0 0 0 0 0</pose>
+    <inertial>
+      <mass value="1.0"/>
+      <origin xyz="0 0 0" rpy="0 0 0"/>
+      <inertia ixx="0.1" ixy="0" ixz="0" iyy="0.1" iyz="0" izz="0.1"/>
+    </inertial>
+    <collision name="front_right_tire_collision">
+      <origin xyz="0 0 0" rpy="0 0 0"/>
+      <geometry>
+        <mesh scale="0.001 0.001 0.001" filename="package://digital_twin/meshes/tire.stl"/>
+      </geometry>
+    </collision>
+    <visual name="front_right_tire_visual">
+      <origin xyz="0 0 0" rpy="0 0 0"/>
+      <geometry>
+        <mesh scale="0.001 0.001 0.001" filename="package://digital_twin/meshes/tire.stl"/>
+      </geometry>
+    </visual>
+  </link>
+  <!-- LINK: front_right_disk -->
+  <link name="front_right_disk">
+    <pose>0 0 0 0 0 0</pose>
+    <collision name="front_right_disk_collision">
+      <origin xyz="0 0 0" rpy="0 0 0"/>
+      <geometry>
+        <mesh scale="0.001 0.001 0.001" filename="package://digital_twin/meshes/disk.stl"/>
+      </geometry>
+    </collision>
+    <visual name="front_right_disk_visual">
+      <origin xyz="0 0 0" rpy="0 0 0"/>
+      <geometry>
+        <mesh scale="0.001 0.001 0.001" filename="package://digital_twin/meshes/disk.stl"/>
       </geometry>
     </visual>
@@ -60,4 +298,12 @@
     <material>Gazebo/Green</material>
   </gazebo>
+  <!-- COLOR: left_steer -->
+  <gazebo reference="left_steer">
+    <material>Gazebo/Grey</material>
+  </gazebo>
+  <!-- COLOR: right_steer -->
+  <gazebo reference="right_steer">
+    <material>Gazebo/Grey</material>
+  </gazebo>
   <!-- COLOR: board -->
   <gazebo reference="board">
@@ -67,4 +313,48 @@
   <gazebo reference="rpi">
     <material>Gazebo/Green</material>
+  </gazebo>
+  <!-- COLOR: motor1 -->
+  <gazebo reference="motor1">
+    <material>Gazebo/Grey</material>
+  </gazebo>
+  <!-- COLOR: motor2 -->
+  <gazebo reference="motor2">
+    <material>Gazebo/Grey</material>
+  </gazebo>
+  <!-- COLOR: cover -->
+  <gazebo reference="cover">
+    <material>Gazebo/GreenGlow</material>
+  </gazebo>
+  <!-- COLOR: rear_left_tire -->
+  <gazebo reference="rear_left_tire">
+    <material>Gazebo/DarkGrey</material>
+  </gazebo>
+  <!-- COLOR: rear_left_disk -->
+  <gazebo reference="rear_left_disk">
+    <material>Gazebo/Blue</material>
+  </gazebo>
+  <!-- COLOR: rear_right_tire -->
+  <gazebo reference="rear_right_tire">
+    <material>Gazebo/DarkGrey</material>
+  </gazebo>
+  <!-- COLOR: rear_right_disk -->
+  <gazebo reference="rear_right_disk">
+    <material>Gazebo/Blue</material>
+  </gazebo>
+  <!-- COLOR: front_left_tire -->
+  <gazebo reference="front_left_tire">
+    <material>Gazebo/DarkGrey</material>
+  </gazebo>
+  <!-- COLOR: front_left_disk -->
+  <gazebo reference="front_left_disk">
+    <material>Gazebo/Blue</material>
+  </gazebo>
+  <!-- COLOR: front_right_tire -->
+  <gazebo reference="front_right_tire">
+    <material>Gazebo/DarkGrey</material>
+  </gazebo>
+  <!-- COLOR: front_right_disk -->
+  <gazebo reference="front_right_disk">
+    <material>Gazebo/Blue</material>
   </gazebo>
   <!-- JOINT: chassis -->
@@ -74,4 +364,22 @@
     <child link="chassis"/>
   </joint>
+  <!-- JOINT: left_steer -->
+  <joint name="left_steer_joint" type="continuous">
+    <origin xyz="0.179 0.060 0.013" rpy="0 0 0"/>
+    <parent link="chassis"/>
+    <child link="left_steer"/>
+    <axis xyz="0 0 1" rpy="0 0 0"/>
+    <limit effort="10000" velocity="1000"/>
+    <dynamics damping="1.0" friction="1.0"/>
+  </joint>
+  <!-- JOINT: right_steer -->
+  <joint name="right_steer_joint" type="continuous">
+    <origin xyz="0.179 -0.060 0.013" rpy="0 0 0"/>
+    <parent link="chassis"/>
+    <child link="right_steer"/>
+    <axis xyz="0 0 1" rpy="0 0 0"/>
+    <limit effort="10000" velocity="1000"/>
+    <dynamics damping="1.0" friction="1.0"/>
+  </joint>
   <!-- JOINT: board -->
   <joint name="board_joint" type="fixed">
@@ -86,3 +394,81 @@
     <child link="rpi"/>
   </joint>
+  <!-- JOINT: motor1 -->
+  <joint name="motor1_joint" type="fixed">
+    <origin xyz="0.024 0.047 0.023" rpy="1.570796 0 0"/>
+    <parent link="chassis"/>
+    <child link="motor1"/>
+  </joint>
+  <!-- JOINT: motor2 -->
+  <joint name="motor2_joint" type="fixed">
+    <origin xyz="0.024 -0.047 0.023" rpy="1.570796 0 0"/>
+    <parent link="chassis"/>
+    <child link="motor2"/>
+  </joint>
+  <!-- JOINT: cover -->
+  <joint name="cover_joint" type="fixed">
+    <origin xyz="0.024 0 0.023" rpy="1.570796 0 0"/>
+    <parent link="chassis"/>
+    <child link="cover"/>
+  </joint>
+  <!-- JOINT: rear_left_tire -->
+  <joint name="rear_left_tire_joint" type="continuous">
+    <origin xyz="0.024 0.0855 0.015" rpy="1.570796 0 0"/>
+    <parent link="chassis"/>
+    <child link="rear_left_tire"/>
+    <axis xyz="0 1 0" rpy="0 0 0"/>
+    <limit effort="10000" velocity="1000"/>
+    <dynamics damping="1.0" friction="1.0"/>
+  </joint>
+  <!-- JOINT: rear_left_disk -->
+  <joint name="rear_left_disk_joint" type="fixed">
+    <origin xyz="0 0 0" rpy="-3.141592 0 0"/>
+    <parent link="rear_left_tire"/>
+    <child link="rear_left_disk"/>
+  </joint>
+  <!-- JOINT: rear_right_tire -->
+  <joint name="rear_right_tire_joint" type="continuous">
+    <origin xyz="0.024 -0.0855 0.015" rpy="1.570796 0 0"/>
+    <parent link="chassis"/>
+    <child link="rear_right_tire"/>
+    <axis xyz="0 1 0" rpy="0 0 0"/>
+    <limit effort="10000" velocity="1000"/>
+    <dynamics damping="1.0" friction="1.0"/>
+  </joint>
+  <!-- JOINT: rear_right_disk -->
+  <joint name="rear_right_disk_joint" type="fixed">
+    <origin xyz="0 0 0" rpy="0 0 0"/>
+    <parent link="rear_right_tire"/>
+    <child link="rear_right_disk"/>
+  </joint>
+  <!-- JOINT: front_left_tire -->
+  <joint name="front_left_tire_joint" type="continuous">
+    <origin xyz="0 0.014 0.002" rpy="1.570796 0 0"/>
+    <parent link="left_steer"/>
+    <child link="front_left_tire"/>
+    <axis xyz="0 1 0" rpy="0 0 0"/>
+    <limit effort="10000" velocity="1000"/>
+    <dynamics damping="1.0" friction="1.0"/>
+  </joint>
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
Commit message: #8 Piracer not going forward

File: piracer_ws/src/digital_twin/description/piracer.xacro (robot description, xacro)
@@ -7,5 +7,5 @@
     <pose>0 0 0 0 0 0</pose>
     <inertial>
-      <mass value="10.0"/>
+      <mass value="1.0"/>
       <origin xyz="0.118 0 0" rpy="0 0 0"/>
       <inertia ixx="0.1" ixy="0" ixz="0" iyy="0.1" iyz="0" izz="0.1"/>
@@ -21,4 +21,25 @@
       <geometry>
         <mesh scale="0.001 0.001 0.001" filename="package://digital_twin/meshes/chassis.stl"/>
+      </geometry>
+    </visual>
+  </link>
+  <!-- LINK: main_steer -->
+  <link name="main_steer">
+    <pose>0 0 0 0 0 0</pose>
+    <inertial>
+      <mass value="0.1"/>
+      <origin xyz="0 0 0" rpy="0 0 0"/>
+      <inertia ixx="0.1" ixy="0" ixz="0" iyy="0.1" iyz="0" izz="0.1"/>
+    </inertial>
+    <collision name="main_steer_collision">
+      <origin xyz="0 0 0" rpy="0 0 0"/>
+      <geometry>
+        <cylinder length="0.010" radius="0.010"/>
+      </geometry>
+    </collision>
+    <visual name="main_steer_visual">
+      <origin xyz="0 0 0" rpy="0 0 0"/>
+      <geometry>
+        <cylinder length="0.010" radius="0.010"/>
       </geometry>
     </visual>
@@ -297,4 +318,8 @@
   <gazebo reference="chassis">
     <material>Gazebo/Green</material>
+  </gazebo>
+  <!-- COLOR: main_steer -->
+  <gazebo reference="main_steer">
+    <material>Gazebo/Grey</material>
   </gazebo>
   <!-- COLOR: left_steer -->
@@ -364,4 +389,13 @@
     <child link="chassis"/>
   </joint>
+  <!-- JOINT: main_steer -->
+  <joint name="main_steer_joint" type="continuous">
+    <origin xyz="0.170 0 0.013" rpy="0 0 0"/>
+    <parent link="chassis"/>
+    <child link="main_steer"/>
+    <axis xyz="0 0 1" rpy="0 0 0"/>
+    <limit effort="10000" velocity="1000"/>
+    <dynamics damping="1.0" friction="1.0"/>
+  </joint>
   <!-- JOINT: left_steer -->
   <joint name="left_steer_joint" type="continuous">
@@ -417,5 +451,5 @@
     <parent link="chassis"/>
     <child link="rear_left_tire"/>
-    <axis xyz="0 1 0" rpy="0 0 0"/>
+    <axis xyz="0 0 1" rpy="0 0 0"/>
     <limit effort="10000" velocity="1000"/>
     <dynamics damping="1.0" friction="1.0"/>
@@ -432,5 +466,5 @@
     <parent link="chassis"/>
     <child link="rear_right_tire"/>
-    <axis xyz="0 1 0" rpy="0 0 0"/>
+    <axis xyz="0 0 1" rpy="0 0 0"/>
     <limit effort="10000" velocity="1000"/>
     <dynamics damping="1.0" friction="1.0"/>
@@ -447,5 +481,5 @@
     <parent link="left_steer"/>
     <child link="front_left_tire"/>
-    <axis xyz="0 1 0" rpy="0 0 0"/>
+    <axis xyz="0 0 1" rpy="0 0 0"/>
     <limit effort="10000" velocity="1000"/>
     <dynamics damping="1.0" friction="1.0"/>
@@ -462,5 +496,5 @@
     <parent link="right_steer"/>
     <child link="front_right_tire"/>
-    <axis xyz="0 1 0" rpy="0 0 0"/>
+    <axis xyz="0 0 1" rpy="0 0 0"/>
     <limit effort="10000" velocity="1000"/>
     <dynamics damping="1.0" friction="1.0"/>
@@ -472,3 +506,37 @@
     <child link="front_right_disk"/>
   </joint>
+  <!-- PLUGIN: drive -->
+  <gazebo>
+    <plugin name="ackermann_drive_controller" filename="libgazebo_ros_ackermann_drive.so">
+      <ros>
+        <namespace>/piracer</namespace>
+        <argument>/cmd_vel:=cmd_vel</argument>
+        <argument>/odom:=odom</argument>
+        <argument>/distance:=distance</argument>
+      </ros>
+      <update_rate>100.0</update_rate>
+      <odometry_frame>odom</odometry_frame>
+      <robot_base_frame>base_footprint</robot_base_frame>
+      <front_left_joint>front_left_tire_joint</front_left_joint>
+      <front_right_joint>front_right_tire_joint</front_right_joint>
+      <rear_left_joint>rear_left_tire_joint</rear_left_joint>
+      <rear_right_joint>rear_right_tire_joint</rear_right_joint>
+      <left_steering_joint>left_steer_joint</left_steering_joint>
+      <right_steering_joint>right_steer_joint</right_steering_joint>
+      <steering_wheel_joint>main_steer_joint</steering_wheel_joint>
+      <max_steer>0.6458</max_steer>
+      <max_steering_angle>7.85</max_steering_angle>
+      <max_speed>100</max_speed>
+      <left_steering_pid_gain>1500 0 1</left_steering_pid_gain>
+      <left_steering_i_range>0 0</left_steering_i_range>
+      <right_steering_pid_gain>1500 0 1</right_steering_pid_gain>
+      <right_steering_i_range>0 0</right_steering_i_range>
+      <linear_velocity_pid_gain>10 0 1</linear_velocity_pid_gain>
+      <linear_velocity_i_range>0 0</linear_velocity_i_range>
+      <publish_odom>true</publish_odom>
+      <publish_odom_tf>true</publish_odom_tf>
+      <publish_wheel_tf>false</publish_wheel_tf>
+      <publish_distance>false</publish_distance>
+    </plugin>
+  </gazebo>
 </robot>

Commit message: #8 Piracer operates normally

File: piracer_ws/src/digital_twin/description/piracer.xacro (robot description, xacro)
@@ -7,5 +7,5 @@
     <pose>0 0 0 0 0 0</pose>
     <inertial>
-      <mass value="1.0"/>
+      <mass value="1000.0"/>
       <origin xyz="0.118 0 0" rpy="0 0 0"/>
       <inertia ixx="0.1" ixy="0" ixz="0" iyy="0.1" iyz="0" izz="0.1"/>
@@ -28,5 +28,5 @@
     <pose>0 0 0 0 0 0</pose>
     <inertial>
-      <mass value="0.1"/>
+      <mass value="1.0"/>
       <origin xyz="0 0 0" rpy="0 0 0"/>
       <inertia ixx="0.1" ixy="0" ixz="0" iyy="0.1" iyz="0" izz="0.1"/>
@@ -49,5 +49,5 @@
     <pose>0 0 0 0 0 0</pose>
     <inertial>
-      <mass value="0.1"/>
+      <mass value="1.0"/>
       <origin xyz="0 0 0" rpy="0 0 0"/>
       <inertia ixx="0.1" ixy="0" ixz="0" iyy="0.1" iyz="0" izz="0.1"/>
@@ -70,5 +70,5 @@
     <pose>0 0 0 0 0 0</pose>
     <inertial>
-      <mass value="0.1"/>
+      <mass value="1.0"/>
       <origin xyz="0 0 0" rpy="0 0 0"/>
       <inertia ixx="0.1" ixy="0" ixz="0" iyy="0.1" iyz="0" izz="0.1"/>
@@ -171,5 +171,5 @@
     <pose>0 0 0 0 0 0</pose>
     <inertial>
-      <mass value="1.0"/>
+      <mass value="50.0"/>
       <origin xyz="0 0 0" rpy="0 0 0"/>
       <inertia ixx="0.1" ixy="0" ixz="0" iyy="0.1" iyz="0" izz="0.1"/>
@@ -178,5 +178,5 @@
       <origin xyz="0 0 0" rpy="0 0 0"/>
       <geometry>
-        <mesh scale="0.001 0.001 0.001" filename="package://digital_twin/meshes/tire.stl"/>
+        <cylinder length="0.026" radius="0.034"/>
       </geometry>
     </collision>
@@ -208,5 +208,5 @@
     <pose>0 0 0 0 0 0</pose>
     <inertial>
-      <mass value="1.0"/>
+      <mass value="50.0"/>
       <origin xyz="0 0 0" rpy="0 0 0"/>
       <inertia ixx="0.1" ixy="0" ixz="0" iyy="0.1" iyz="0" izz="0.1"/>
@@ -215,5 +215,5 @@
       <origin xyz="0 0 0" rpy="0 0 0"/>
       <geometry>
-        <mesh scale="0.001 0.001 0.001" filename="package://digital_twin/meshes/tire.stl"/>
+        <cylinder length="0.026" radius="0.034"/>
       </geometry>
     </collision>
@@ -245,5 +245,5 @@
     <pose>0 0 0 0 0 0</pose>
     <inertial>
-      <mass value="1.0"/>
+      <mass value="50.0"/>
       <origin xyz="0 0 0" rpy="0 0 0"/>
       <inertia ixx="0.1" ixy="0" ixz="0" iyy="0.1" iyz="0" izz="0.1"/>
@@ -282,5 +282,5 @@
     <pose>0 0 0 0 0 0</pose>
     <inertial>
-      <mass value="1.0"/>
+      <mass value="50.0"/>
       <origin xyz="0 0 0" rpy="0 0 0"/>
       <inertia ixx="0.1" ixy="0" ixz="0" iyy="0.1" iyz="0" izz="0.1"/>
@@ -337,5 +337,5 @@
   <!-- COLOR: rpi -->
   <gazebo reference="rpi">
-    <material>Gazebo/Green</material>
+    <material>Gazebo/GreenTransparent</material>
   </gazebo>
   <!-- COLOR: motor1 -->
@@ -448,5 +448,5 @@
   <!-- JOINT: rear_left_tire -->
   <joint name="rear_left_tire_joint" type="continuous">
-    <origin xyz="0.024 0.0855 0.015" rpy="1.570796 0 0"/>
+    <origin xyz="0.024 0.0855 0.015" rpy="-1.570796 0 0"/>
     <parent link="chassis"/>
     <child link="rear_left_tire"/>
@@ -463,5 +463,5 @@
   <!-- JOINT: rear_right_tire -->
   <joint name="rear_right_tire_joint" type="continuous">
-    <origin xyz="0.024 -0.0855 0.015" rpy="1.570796 0 0"/>
+    <origin xyz="0.024 -0.0855 0.015" rpy="-1.570796 0 0"/>
     <parent link="chassis"/>
     <child link="rear_right_tire"/>
@@ -525,10 +525,10 @@
       <right_steering_joint>right_steer_joint</right_steering_joint>
       <steering_wheel_joint>main_steer_joint</steering_wheel_joint>
-      <max_steer>0.6458</max_steer>
-      <max_steering_angle>7.85</max_steering_angle>
+      <max_steer>0.3</max_steer>
+      <max_steering_angle>5.0</max_steering_angle>
       <max_speed>100</max_speed>
-      <left_steering_pid_gain>1500 0 1</left_steering_pid_gain>
+      <left_steering_pid_gain>1000 0 1</left_steering_pid_gain>
       <left_steering_i_range>0 0</left_steering_i_range>
-      <right_steering_pid_gain>1500 0 1</right_steering_pid_gain>
+      <right_steering_pid_gain>1000 0 1</right_steering_pid_gain>
       <right_steering_i_range>0 0</right_steering_i_range>
       <linear_velocity_pid_gain>10 0 1</linear_velocity_pid_gain>
