Commit message: a

File: sim_ws/src/sim/description/piracer.xacro (robot description, xacro)
@@ -14,5 +14,5 @@
       <origin xyz="0 0 0" rpy="0 0 0"/>
       <geometry>
-        <mesh scale="0.001 0.001 0.001" filename="package://digital_twin/meshes/chassis.stl"/>
+        <mesh scale="0.001 0.001 0.001" filename="package://sim/meshes/chassis.stl"/>
       </geometry>
     </collision>
@@ -20,5 +20,5 @@
       <origin xyz="0 0 0" rpy="0 0 0"/>
       <geometry>
-        <mesh scale="0.001 0.001 0.001" filename="package://digital_twin/meshes/chassis.stl"/>
+        <mesh scale="0.001 0.001 0.001" filename="package://sim/meshes/chassis.stl"/>
       </geometry>
     </visual>
@@ -93,5 +93,5 @@
       <origin xyz="0 0 0" rpy="0 0 0"/>
       <geometry>
-        <mesh scale="0.001 0.001 0.001" filename="package://digital_twin/meshes/board.stl"/>
+        <mesh scale="0.001 0.001 0.001" filename="package://sim/meshes/board.stl"/>
       </geometry>
     </collision>
@@ -99,5 +99,5 @@
       <origin xyz="0 0 0" rpy="0 0 0"/>
       <geometry>
-        <mesh scale="0.001 0.001 0.001" filename="package://digital_twin/meshes/board.stl"/>
+        <mesh scale="0.001 0.001 0.001" filename="package://sim/meshes/board.stl"/>
       </geometry>
     </visual>
@@ -109,5 +109,5 @@
       <origin xyz="0 0 0" rpy="0 0 0"/>
       <geometry>
-        <mesh scale="0.001 0.001 0.001" filename="package://digital_twin/meshes/rpi.stl"/>
+        <mesh scale="0.001 0.001 0.001" filename="package://sim/meshes/rpi.stl"/>
       </geometry>
     </collision>
@@ -115,5 +115,5 @@
       <origin xyz="0 0 0" rpy="0 0 0"/>
       <geometry>
-        <mesh scale="0.001 0.001 0.001" filename="package://digital_twin/meshes/rpi.stl"/>
+        <mesh scale="0.001 0.001 0.001" filename="package://sim/meshes/rpi.stl"/>
       </geometry>
     </visual>
@@ -125,5 +125,5 @@
       <origin xyz="0 0 0" rpy="0 0 0"/>
       <geometry>
-        <mesh scale="0.001 0.001 0.001" filename="package://digital_twin/meshes/motor.stl"/>
+        <mesh scale="0.001 0.001 0.001" filename="package://sim/meshes/motor.stl"/>
       </geometry>
     </collision>
@@ -131,5 +131,5 @@
       <origin xyz="0 0 0" rpy="0 0 0"/>
       <geometry>
-        <mesh scale="0.001 0.001 0.001" filename="package://digital_twin/meshes/motor.stl"/>
+        <mesh scale="0.001 0.001 0.001" filename="package://sim/meshes/motor.stl"/>
       </geometry>
     </visual>
@@ -141,5 +141,5 @@
       <origin xyz="0 0 0" rpy="0 0 0"/>
       <geometry>
-        <mesh scale="0.001 0.001 0.001" filename="package://digital_twin/meshes/motor.stl"/>
+        <mesh scale="0.001 0.001 0.001" filename="package://sim/meshes/motor.stl"/>
       </geometry>
     </collision>
@@ -147,5 +147,5 @@
       <origin xyz="0 0 0" rpy="0 0 0"/>
       <geometry>
-        <mesh scale="0.001 0.001 0.001" filename="package://digital_twin/meshes/motor.stl"/>
+        <mesh scale="0.001 0.001 0.001" filename="package://sim/meshes/motor.stl"/>
       </geometry>
     </visual>
@@ -157,5 +157,5 @@
       <origin xyz="0 0 0" rpy="0 0 0"/>
       <geometry>
-        <mesh scale="0.001 0.001 0.001" filename="package://digital_twin/meshes/cover.stl"/>
+        <mesh scale="0.001 0.001 0.001" filename="package://sim/meshes/cover.stl"/>
       </geometry>
     </collision>
@@ -163,5 +163,5 @@
       <origin xyz="0 0 0" rpy="0 0 0"/>
       <geometry>
-        <mesh scale="0.001 0.001 0.001" filename="package://digital_twin/meshes/cover.stl"/>
+        <mesh scale="0.001 0.001 0.001" filename="package://sim/meshes/cover.stl"/>
       </geometry>
     </visual>
@@ -184,5 +184,5 @@
       <origin xyz="0 0 0" rpy="0 0 0"/>
       <geometry>
-        <mesh scale="0.001 0.001 0.001" filename="package://digital_twin/meshes/tire.stl"/>
+        <mesh scale="0.001 0.001 0.001" filename="package://sim/meshes/tire.stl"/>
       </geometry>
     </visual>
@@ -194,5 +194,5 @@
       <origin xyz="0 0 0" rpy="0 0 0"/>
       <geometry>
-        <mesh scale="0.001 0.001 0.001" filename="package://digital_twin/meshes/disk.stl"/>
+        <mesh scale="0.001 0.001 0.001" filename="package://sim/meshes/disk.stl"/>
       </geometry>
     </collision>
@@ -200,5 +200,5 @@
       <origin xyz="0 0 0" rpy="0 0 0"/>
       <geometry>
-        <mesh scale="0.001 0.001 0.001" filename="package://digital_twin/meshes/disk.stl"/>
+        <mesh scale="0.001 0.001 0.001" filename="package://sim/meshes/disk.stl"/>
       </geometry>
     </visual>
@@ -221,5 +221,5 @@
       <origin xyz="0 0 0" rpy="0 0 0"/>
       <geometry>
-        <mesh scale="0.001 0.001 0.001" filename="package://digital_twin/meshes/tire.stl"/>
+        <mesh scale="0.001 0.001 0.001" filename="package://sim/meshes/tire.stl"/>
       </geometry>
     </visual>
@@ -231,5 +231,5 @@
       <origin xyz="0 0 0" rpy="0 0 0"/>
       <geometry>
-        <mesh scale="0.001 0.001 0.001" filename="package://digital_twin/meshes/disk.stl"/>
+        <mesh scale="0.001 0.001 0.001" filename="package://sim/meshes/disk.stl"/>
       </geometry>
     </collision>
@@ -237,5 +237,5 @@
       <origin xyz="0 0 0" rpy="0 0 0"/>
       <geometry>
-        <mesh scale="0.001 0.001 0.001" filename="package://digital_twin/meshes/disk.stl"/>
+        <mesh scale="0.001 0.001 0.001" filename="package://sim/meshes/disk.stl"/>
       </geometry>
     </visual>
@@ -252,5 +252,5 @@
       <origin xyz="0 0 0" rpy="0 0 0"/>
       <geometry>
-        <mesh scale="0.001 0.001 0.001" filename="package://digital_twin/meshes/tire.stl"/>
+        <mesh scale="0.001 0.001 0.001" filename="package://sim/meshes/tire.stl"/>
       </geometry>
     </collision>
@@ -258,5 +258,5 @@
       <origin xyz="0 0 0" rpy="0 0 0"/>
       <geometry>
-        <mesh scale="0.001 0.001 0.001" filename="package://digital_twin/meshes/tire.stl"/>
+        <mesh scale="0.001 0.001 0.001" filename="package://sim/meshes/tire.stl"/>
       </geometry>
     </visual>
@@ -268,5 +268,5 @@
       <origin xyz="0 0 0" rpy="0 0 0"/>
       <geometry>
-        <mesh scale="0.001 0.001 0.001" filename="package://digital_twin/meshes/disk.stl"/>
+        <mesh scale="0.001 0.001 0.001" filename="package://sim/meshes/disk.stl"/>
       </geometry>
     </collision>
@@ -274,5 +274,5 @@
       <origin xyz="0 0 0" rpy="0 0 0"/>
       <geometry>
-        <mesh scale="0.001 0.001 0.001" filename="package://digital_twin/meshes/disk.stl"/>
+        <mesh scale="0.001 0.001 0.001" filename="package://sim/meshes/disk.stl"/>
       </geometry>
     </visual>
@@ -289,5 +289,5 @@
       <origin xyz="0 0 0" rpy="0 0 0"/>
       <geometry>
-        <mesh scale="0.001 0.001 0.001" filename="package://digital_twin/meshes/tire.stl"/>
+        <mesh scale="0.001 0.001 0.001" filename="package://sim/meshes/tire.stl"/>
       </geometry>
     </collision>
@@ -295,5 +295,5 @@
       <origin xyz="0 0 0" rpy="0 0 0"/>
       <geometry>
-        <mesh scale="0.001 0.001 0.001" filename="package://digital_twin/meshes/tire.stl"/>
+        <mesh scale="0.001 0.001 0.001" filename="package://sim/meshes/tire.stl"/>
       </geometry>
     </visual>
@@ -305,5 +305,5 @@
       <origin xyz="0 0 0" rpy="0 0 0"/>
       <geometry>
-        <mesh scale="0.001 0.001 0.001" filename="package://digital_twin/meshes/disk.stl"/>
+        <mesh scale="0.001 0.001 0.001" filename="package://sim/meshes/disk.stl"/>
       </geometry>
     </collision>
@@ -311,5 +311,5 @@
       <origin xyz="0 0 0" rpy="0 0 0"/>
       <geometry>
-        <mesh scale="0.001 0.001 0.001" filename="package://digital_twin/meshes/disk.stl"/>
+        <mesh scale="0.001 0.001 0.001" filename="package://sim/meshes/disk.stl"/>
       </geometry>
     </visual>

Commit message: a

File: sim_ws/src/sim/description/piracer.xacro (robot description, xacro)
@@ -252,5 +252,5 @@
       <origin xyz="0 0 0" rpy="0 0 0"/>
       <geometry>
-        <mesh scale="0.001 0.001 0.001" filename="package://sim/meshes/tire.stl"/>
+        <cylinder length="0.026" radius="0.034"/>
       </geometry>
     </collision>
@@ -289,5 +289,5 @@
       <origin xyz="0 0 0" rpy="0 0 0"/>
       <geometry>
-        <mesh scale="0.001 0.001 0.001" filename="package://sim/meshes/tire.stl"/>
+        <cylinder length="0.026" radius="0.034"/>
       </geometry>
     </collision>
@@ -312,4 +312,20 @@
       <geometry>
         <mesh scale="0.001 0.001 0.001" filename="package://sim/meshes/disk.stl"/>
+      </geometry>
+    </visual>
+  </link>
+  <!-- LINK: camera -->
+  <link name='camera'>
+    <pose>0 0 0 0 0 0</pose>
+    <collision name='camera_collision'>
+      <origin xyz="0 0 0" rpy=" 0 0 0"/>
+      <geometry>
+        <box size=".001 .001 .001"/>
+      </geometry>
+    </collision>
+    <visual name='camera_visual'>
+      <origin xyz="0 0 0" rpy=" 0 0 0"/>
+      <geometry>
+        <box size=".001 .001 .001"/>
       </geometry>
     </visual>
@@ -505,4 +521,10 @@
     <parent link="front_right_tire"/>
     <child link="front_right_disk"/>
+  </joint>
+  <!-- JOINT: camera -->
+  <joint name="camera_joint" type="fixed">
+    <origin xyz="0.180 0 0.120" rpy="0 0 0"/>
+    <parent link="chassis"/>
+    <child link="camera"/>
   </joint>
   <!-- PLUGIN: drive -->
@@ -541,5 +563,5 @@
   </gazebo>
   <!-- camera -->
-  <!-- <gazebo reference="camera">
+  <gazebo reference="camera">
     <sensor type="camera" name="camera_sensor">
       <update_rate>30.0</update_rate>
@@ -576,4 +598,4 @@
       </plugin>
     </sensor>
-  </gazebo> -->
+  </gazebo>
 </robot>
